File: Amplifier ECAD/Amplifier Hardware R1.kicad_sch (KiCad schematic)
At the start: 15 parts, among them J1 SJ1-3525N, J2 NMJ6HFD2, J3 NMJ6HFD2, J4 NMJ6HFD2, J5 NMJ6HFD2, J6 NMJ6HFD2, J7 SJ1-3525N

Commit message: Solid polygon connections for holes
Parts:
- H1, H2, H3, H4, H5, H6, H7, H8: value MountingHole_Pad -> M3
Changed lines of the file:
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@@
       (effects (font (size 1.27 1.27)) (justify left))
     )
-    (property "Value" "MountingHole_Pad" (at 273.05 140.97 90)
+    (property "Value" "M3" (at 273.05 140.97 90)
       (effects (font (size 1.27 1.27)) (justify left))
     )
@@
       (effects (font (size 1.27 1.27)) (justify left))
     )
-    (property "Value" "MountingHole_Pad" (at 273.05 87.63 90)
+    (property "Value" "M3" (at 273.05 87.63 90)
       (effects (font (size 1.27 1.27)) (justify left))
     )
@@
       (effects (font (size 1.27 1.27)) (justify left))
     )
-    (property "Value" "MountingHole_Pad" (at 273.05 105.41 90)
+    (property "Value" "M3" (at 273.05 105.41 90)
       (effects (font (size 1.27 1.27)) (justify left))
     )
@@
       (effects (font (size 1.27 1.27)) (justify left))
     )
-    (property "Value" "MountingHole_Pad" (at 273.05 96.52 90)
+    (property "Value" "M3" (at 273.05 96.52 90)
       (effects (font (size 1.27 1.27)) (justify left))
     )
@@
       (effects (font (size 1.27 1.27)) (justify left))
     )
-    (property "Value" "MountingHole_Pad" (at 273.05 149.86 90)
+    (property "Value" "M3" (at 273.05 149.86 90)
       (effects (font (size 1.27 1.27)) (justify left))
     )
@@
       (effects (font (size 1.27 1.27)) (justify left))
     )
-    (property "Value" "MountingHole_Pad" (at 273.05 132.08 90)
+    (property "Value" "M3" (at 273.05 132.08 90)
       (effects (font (size 1.27 1.27)) (justify left))
     )
@@
       (effects (font (size 1.27 1.27)) (justify left))
     )
-    (property "Value" "MountingHole_Pad" (at 273.05 123.19 90)
+    (property "Value" "M3" (at 273.05 123.19 90)
       (effects (font (size 1.27 1.27)) (justify left))
     )
@@
       (effects (font (size 1.27 1.27)) (justify left))
     )
-    (property "Value" "MountingHole_Pad" (at 273.05 114.3 90)
-      (effects (font (size 1.27 1.27)) (justify left))
-    )
+    (property "Value" "M3" (at 273.05 114.3 90)
+      (effects (font (size 1.27 1.27)) (justify left))
+    )
