File: Amplifier ECAD/modamp_AntiAlias.kicad_sch (KiCad schematic)
At the start: 8 parts, among them U3 MCP6004

Commit message: File renaming; updating supplier references
Parts:
- C20, C22: footprint Custom-RLC:C_Disc_L7.2mm_W2.5mm_H6.6mm_P5.00mm_MODIFIED_1 -> Custom-RLC:C_KEMET_C322; symbol Custom-CapacitorTHT:FG28C0G2A472JRT06 -> Custom-CapacitorTHT:C322C472J1G5TA; Manufacturer TDK Corporation -> KEMET; Part Number FG28C0G2A472JRT06 -> C322C472J1G5TA
- C21: footprint Custom-RLC:C_Disc_L7.2mm_W2.5mm_H6.6mm_P5.00mm_MODIFIED_1 -> Custom-RLC:C_KEMET_C317; symbol Custom-CapacitorTHT:FG28C0G1H471JNT06 -> Custom-CapacitorTHT:C317C471J1G5TA; Manufacturer TDK Corporation -> KEMET; Part Number FG28C0G1H471JNT06 -> C317C471J1G5TA
- R17, R18, R19: symbol Custom-ResistorTHT:MFR-25FRF52-10K -> Custom-ResistorTHT:CF14JT10K0; Manufacturer YAGEO -> Stackpole Electronics Inc; Part Number MFR-25FRF52-10K -> CF14JT10K0
- R?: symbol Custom-ResistorTHT:MFR-25FRF52-3K3 -> Custom-ResistorTHT:CF14JT3K30; Manufacturer YAGEO -> Stackpole Electronics Inc; Part Number MFR-25FRF52-3K3 -> CF14JT3K30
