File: Amplifier ECAD/modamp_Channel.kicad_sch (KiCad schematic)
At the start: 8 parts, among them SW2 EC11

Commit message: File renaming; updating supplier references
Parts:
- C31: footprint Custom-RLC:C_Disc_L7.2mm_W2.5mm_H6.6mm_P5.00mm_MODIFIED_1 -> Custom-RLC:C_KEMET_C317; symbol Custom-CapacitorTHT:FG28X7R1H104KNT06 -> Custom-CapacitorTHT:C317C104K5R5TA; Manufacturer TDK Corporation -> KEMET; Part Number FG28X7R1H104KNT06 -> C317C104K5R5TA
- D2: symbol Custom-Optoelectronic:QBL8RGB60D0-2897 -> Custom-Optoelectronic:WP154A4SEJ3VBDZGW/CA; Manufacturer QT Brightek (QTB) -> Kingbright; Part Number QBL8RGB60D0-2897 -> WP154A4SEJ3VBDZGW/CA
- R32, R33, R34, R35, R36: symbol Custom-ResistorTHT:MFR-25FRF52-470R -> Custom-ResistorTHT:CF14JT470R; Manufacturer YAGEO -> Stackpole Electronics Inc; Part Number MFR-25FRF52-470R -> CF14JT470R
