File: Amplifier ECAD/modamp_VolMixOut.kicad_sch (KiCad schematic)
At the start: 17 parts, among them U2 MCP6004

Commit message: File renaming; updating supplier references
Parts:
- C14, C15: footprint Custom-RLC:C_Disc_L7.2mm_W2.5mm_H6.6mm_P5.00mm_MODIFIED_1 -> Custom-RLC:C_KEMET_C322; symbol Custom-CapacitorTHT:FG28C0G2A472JRT06 -> Custom-CapacitorTHT:C322C472J1G5TA; Manufacturer TDK Corporation -> KEMET; Part Number FG28C0G2A472JRT06 -> C322C472J1G5TA
- C? (x4): footprint Custom-RLC:CP_Radial_D6.3mm_H12.5_P2.50mm -> Custom-RLC:CP_KEMET_ESY; symbol Custom-CapacitorTHT:860020473008 -> Custom-CapacitorTHT:ESY107M025AE3AA; Manufacturer Würth Elektronik -> KEMET; Part Number 860020473008 -> ESY107M025AE3AA
- R10, R11, R12, R13, R14, R9: symbol Custom-ResistorTHT:MFR-25FRF52-3K3 -> Custom-ResistorTHT:CF14JT3K30; Manufacturer YAGEO -> Stackpole Electronics Inc; Part Number MFR-25FRF52-3K3 -> CF14JT3K30
- R15, R16: symbol Custom-ResistorTHT:MFR-25FRF52-10K -> Custom-ResistorTHT:CF14JT10K0; Manufacturer YAGEO -> Stackpole Electronics Inc; Part Number MFR-25FRF52-10K -> CF14JT10K0
