File: Amplifier ECAD/modamp_ui.kicad_sch (KiCad schematic)
At the start: 18 parts, among them SW5 EC11, U5 SH1106

Commit message: File renaming; updating supplier references
Parts:
- added J10: SSQ-104-03-T-S, symbol Custom-Connector:SSQ-104-03-T-S
- D5: symbol Custom-Optoelectronic:QBL7R60D -> Custom-Optoelectronic:WP3A8ID; Manufacturer QT Brightek (QTB) -> Kingbright; Part Number QBL7R60D -> WP3A8ID
- D6, D7, D8: value WHITE -> YELLOW; symbol Custom-Optoelectronic:QBL7IW60D-NW -> Custom-Optoelectronic:WP3A8YD; Manufacturer QT Brightek (QTB) -> Kingbright; Part Number QBL7IW60D-NW -> WP3A8YD
- D9: symbol Custom-Optoelectronic:QBL8RGB60D0-2897 -> Custom-Optoelectronic:WP154A4SEJ3VBDZGW/CA; Manufacturer QT Brightek (QTB) -> Kingbright; Part Number QBL8RGB60D0-2897 -> WP154A4SEJ3VBDZGW/CA
- R47, R48, R49, R50, R51, R52, R53: symbol Custom-ResistorTHT:MFR-25FRF52-470R -> Custom-ResistorTHT:CF14JT470R; Manufacturer YAGEO -> Stackpole Electronics Inc; Part Number MFR-25FRF52-470R -> CF14JT470R
- R54, R55: symbol Custom-ResistorTHT:MFR-25FRF52-10K -> Custom-ResistorTHT:CF14JT10K0; Manufacturer YAGEO -> Stackpole Electronics Inc; Part Number MFR-25FRF52-10K -> CF14JT10K0
Connections:
- no-connect marks 0 -> 4
Other:
- moved on the sheet: D5, D6, D7, D8, D9, JP1, JP2, R47, R48, R49, R50, R51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
