File: Amplifier ECAD/Amplifier Hardware RevB.kicad_sch (KiCad schematic)
At the start: 15 parts, among them J1 SJ1-3525N, J2 NMJ6HFD2, J3 NMJ6HFD2, J4 NMJ6HFD2, J5 NMJ6HFD2, J6 NMJ6HFD2, J7 SJ1-3525N

Commit message: File renaming; updating supplier references
Parts:
- J1, J7: value SJ1-3525N -> 3.5mm TRS; symbol Custom-Connector:SJ1-3525N -> Custom-Connector:35RAPC4BHN2; Manufacturer CUI Devices -> Switchcraft Inc.; Part Number SJ1-3525N -> 35RAPC4BHN2

Commit message: Front and rear panel work; renderings on Fusion360
Parts:
- added H10, H11, H12, H13, H14, H9: M2.6, Custom-Mechanical:MountingHole_2.9mm_5.5mm_Ring, symbol Mechanical:MountingHole
- J2, J3, J4, J5, J6: value NMJ6HFD2 -> 1/4" TRS
Other:
- moved on the sheet: H1, H2, H3, H4, H5, H6, H7, H8
